File: Test/_autosave-Tester.kicad_pcb (KiCad board)
At the start: 2 copper layers, 62.2 x 63.6 mm, 55 parts, among them IC1 ATMEGA328-A, P1 7-16v, P3 5vReg, P4 Servo Power, P5 PMW, P6 Analog Port, P7 RS232, P8 Servo Power 1, SW1 SW_PUSH, U1 7805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

Commit message: Finish Layout
Parts:
- IC1: footprint Housings_QFP:LQFP-32_5x5mm_Pitch0.5mm -> Housings_QFP:TQFP-32_7x7mm_Pitch0.8mm
- moved IC1 44.8 mm to (232.2, 75.1)
Routing:
- net (no net): track 51.2 -> 73.3 mm, vias 9 -> 13
- net GND: track 323.2 -> 307.9 mm, vias 13 -> 9
- net +5V: track 84.7 -> 77.9 mm
