File: Test/Tester.kicad_pcb (KiCad board)
At the start: 2 copper layers, 62.2 x 63.6 mm, 55 parts, among them IC1 ATMEGA328-A, P1 7-16v, P3 5vReg, P4 Servo Power, P5 PMW, P6 Analog Port, P7 RS232, P8 Servo Power 1, SW1 SW_PUSH, U1 7805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

Commit message: Add connections, Add board marks
Routing:
- net +5V: track 73.4 -> 100.9 mm, vias 5 -> 9
- net GND: track 317.4 -> 326.5 mm, vias 13 -> 15
Other:
- board text added: "M A V R I C Main Board Rev1.0 Danny Mallek"
Changed lines of the file:
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@@
   (general
     (links 143)
-    (no_connects 4)
+    (no_connects 1)
     (area 149.022999 32.436999 211.403001 96.214001)
     (thickness 1.6)
-    (drawings 22)
-    (tracks 594)
+    (drawings 23)
+    (tracks 621)
     (zones 0)
     (modules 55)
@@
   )
   (setup
-    (last_trace_width 0.75)
+    (last_trace_width 0.25)
     (user_trace_width 0.05)
     (user_trace_width 0.1)
@@
     (descr "Through hole pin header")
     (tags "pin header")
-    (fp_text reference P8 (at 0 -5.1 90) (layer F.SilkS)
+    (fp_text reference P8 (at 0.0508 -2.5146 90) (layer F.SilkS)
       (effects (font (size 1 1) (thickness 0.15)))
     )
@@
     (descr "Through hole pin header")
     (tags "pin header")
-    (fp_text reference P5 (at 0 -5.1 90) (layer F.SilkS)
+    (fp_text reference P5 (at -0.1016 -2.2606 90) (layer F.SilkS)
       (effects (font (size 1 1) (thickness 0.15)))
     )
@@
     )
   )
+  (gr_text "M A V R I C\nMain Board Rev1.0\nDanny Mallek" (at 160.782 87.2744) (layer F.SilkS)
+    (effects (font (size 1.5 1.5) (thickness 0.1)))
+  )
   (gr_line (start 209.804 96.139) (end 211.328 96.139) (angle 90) (layer Edge.Cuts) (width 0.15))
   (gr_line (start 209.804 32.512) (end 211.328 32.512) (angle 90) (layer Edge.Cuts) (width 0.15))
@@
   (segment (start 162.052 59.7535) (end 166.8145 59.7535) (width 1.25) (layer F.Cu) (net 1))
   (segment (start 158.56966 63.881) (end 158.56966 63.23584) (width 1.25) (layer F.Cu) (net 1) (status 30))
+  (segment (start 197.358 62.77) (end 203.6252 62.77) (width 0.25) (layer F.Cu) (net 2) (status 400000))
+  (segment (start 205.994 63.3476) (end 206.1464 63.3476) (width 0.25) (layer F.Cu) (net 2))
+  (segment (start 205.9432 63.2968) (end 205.994 63.3476) (width 0.25) (layer F.Cu) (net 2))
+  (via (at 205.9432 63.2968) (size 0.6) (drill 0.4) (layers F.Cu B.Cu) (net 2))
+  (segment (start 204.216 63.2968) (end 205.9432 63.2968) (width 0.25) (layer B.Cu) (net 2))
+  (segment (start 203.6572 62.738) (end 204.216 63.2968) (width 0.25) (layer B.Cu) (net 2))
+  (via (at 203.6572 62.738) (size 0.6) (drill 0.4) (layers F.Cu B.Cu) (net 2))
+  (segment (start 203.6252 62.77) (end 203.6572 62.738) (width 0.25) (layer F.Cu) (net 2))
   (via (at 185.5216 86.4616) (size 0.6) (drill 0.4) (layers F.Cu B.Cu) (net 2))
   (segment (start 190.627 83.82) (end 188.1632 83.82) (width 0.75) (layer F.Cu) (net 2) (status 400000))
@@
   (segment (start 164.56914 63.881) (end 167.47236 63.881) (width 1.25) (layer F.Cu) (net 2) (status 10))
   (segment (start 167.47236 63.881) (end 169.545 61.80836) (width 1.25) (layer F.Cu) (net 2))
+  (segment (start 191.9224 89.5604) (end 191.9224 92.1512) (width 0.25) (layer F.Cu) (net 3))
+  (segment (start 203.454 91.2876) (end 203.454 89.8652) (width 0.25) (layer F.Cu) (net 3))
+  (segment (start 202.8952 91.8464) (end 203.454 91.2876) (width 0.25) (layer F.Cu) (net 3))
+  (segment (start 195.072 91.8464) (end 202.8952 91.8464) (width 0.25) (layer F.Cu) (net 3))
+  (segment (start 194.4116 92.5068) (end 195.072 91.8464) (width 0.25) (layer F.Cu) (net 3))
+  (via (at 194.4116 92.5068) (size 0.6) (drill 0.4) (layers F.Cu B.Cu) (net 3))
+  (segment (start 192.278 92.5068) (end 194.4116 92.5068) (width 0.25) (layer B.Cu) (net 3))
+  (via (at 192.278 92.5068) (size 0.6) (drill 0.4) (layers F.Cu B.Cu) (net 3))
+  (segment (start 191.9224 92.1512) (end 192.278 92.5068) (width 0.25) (layer F.Cu) (net 3))
+  (segment (start 192.4685 64.76746) (end 192.4685 62.9031) (width 0.25) (layer F.Cu) (net 3) (status 400000))
+  (segment (start 199.0306 60.3504) (end 200.199 59.182) (width 0.25) (layer F.Cu) (net 3) (status 800000))
+  (segment (start 195.8848 60.3504) (end 199.0306 60.3504) (width 0.25) (layer F.Cu) (net 3))
+  (segment (start 195.6308 60.0964) (end 195.8848 60.3504) (width 0.25) (layer F.Cu) (net 3))
+  (via (at 195.6308 60.0964) (size 0.6) (drill 0.4) (layers F.Cu B.Cu) (net 3))
+  (segment (start 195.2752 60.0964) (end 195.6308 60.0964) (width 0.25) (layer B.Cu) (net 3))
+  (segment (start 192.7352 62.6364) (end 195.2752 60.0964) (width 0.25) (layer B.Cu) (net 3))
+  (via (at 192.7352 62.6364) (size 0.6) (drill 0.4) (layers F.Cu B.Cu) (net 3))
+  (segment (start 192.4685 62.9031) (end 192.7352 62.6364) (width 0.25) (layer F.Cu) (net 3))
   (segment (start 200.199 56.769) (end 199.4662 56.769) (width 0.5) (layer F.Cu) (net 3))
   (segment (start 199.4662 56.769) (end 199.0852 56.388) (width 0.5) (layer F.Cu) (net 3))
@@
   (segment (start 189.357 45.339) (end 190.1952 46.1772) (width 1) (layer F.Cu) (net 3))
   (segment (start 190.1952 46.1772) (end 190.961 46.943) (width 1) (layer F.Cu) (net 3))
+  (segment (start 192.4685 67.05854) (end 197.06946 67.05854) (width 0.25) (layer F.Cu) (net 4) (status C00000))
+  (segment (start 197.06946 67.05854) (end 197.358 66.77) (width 0.25) (layer F.Cu) (net 4) (status C00000))
   (segment (start 192.4685 67.05854) (end 191.46266 67.05854) (width 0.2) (layer F.Cu) (net 4))
   (segment (start 191.46266 67.05854) (end 190.7032 67.818) (width 0.2) (layer F.Cu) (net 4))
@@
   (segment (start 190.7032 67.818) (end 190.6524 67.8688) (width 0.2) (layer B.Cu) (net 4))
   (via (at 190.7032 67.818) (size 0.6) (drill 0.4) (layers F.Cu B.Cu) (net 4))
-  (segment (start 192.4685 67.05854) (end 197.06946 67.05854) (width 0.2) (layer F.Cu) (net 4))
   (segment (start 197.06946 67.05854) (end 197.358 66.77) (width 0.2) (layer F.Cu) (net 4))
   (segment (start 184.1385 75.799) (end 177.74952 75.799) (width 0.25) (layer F.Cu) (net 5))

Commit message: Create Analog Sensor Board, Add Conglomerate1 Board (Advanced Circuits Order)
Parts:
- added C10: 100n, Capacitors_SMD:C_1206, B.Cu at (194.1, 79.5)
- added C11: 100n, Capacitors_SMD:C_1206, B.Cu at (182.2, 71.6)
- added C9: 4.7u, Capacitors_SMD:C_1206, B.Cu at (179.7, 77.6)
- IC1: footprint Housings_QFP:LQFP-32_5x5mm_Pitch0.5mm -> Housings_QFP:TQFP-32_7x7mm_Pitch0.8mm
- moved P3 17.4 mm to (207.6, 80.3), turned to 270 degrees
- moved IC1 3.16 mm to (186.6, 77.6)
- moved P5 0.51 mm to (173.1, 91.7)
Routing:
- net +5V: track 100.9 -> 140.1 mm, vias 9 -> 11
- net /DIO2: track 0.00 -> 25.3 mm, vias 0 -> 2
- net /DIO0: track 27.3 -> 16.9 mm, vias 1 -> 2
- net /~RESET: track 57.9 -> 67.2 mm, vias 3 -> 4
- net /DIO3: track 22.2 -> 13.7 mm
- net GND: track 326.5 -> 320.7 mm, vias 15 -> 9
- net /ADC3: track 29.9 -> 35.5 mm, vias 1 -> 0
- net Net-(C3-Pad1): track 34.5 -> 30.1 mm, vias 4 -> 2
- net (no net): track 31.8 -> 35.9 mm, vias 5 -> 7
- net /7.4v: track 141.4 -> 145.5 mm
- net /PWM2/B: track 18.7 -> 22.3 mm, vias 2 -> 1
- net /MOSI: track 23.3 -> 20.1 mm, vias 0 -> 2
- net /OSC2: track 10.7 -> 7.47 mm
- net /TX: track 4.44 -> 7.38 mm
- net /PMW0/A: track 19.8 -> 17.0 mm, vias 2 -> 0
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Other:
- board text added: "+"
- board text added: "-"
- board text added: "~"
- board text added: "~~"
