File: Test/Tester.sch (KiCad schematic (older format))
At the start: 50 parts, among them IC1 ATMEGA328-A, P1 7-16v, P10 PWM0, P11 PWM1, P12 PWM2, P13 PWM3, P14 PWM4, P15 PWM5, P16 PWM6, P17 PWM7, P18 PWM8, P19 PWM9, P2 7-16V, P20 PWM10, P21 PWM11, P22 PWM12, P23 PWM13, P24 PWM14, P25 PWM15, P26 I2C BUS, P27 ISP, P3 5vReg, P4 Servo Power, P5 PMW, P6 Analog Port, P7 RS232, P8 Servo Power 1, P9 DIO Port, SW1 SW_PUSH, U1 7805, X1 16MHz

Commit message: Finish Layout
Parts:
- IC1: footprint Housings_QFP:LQFP-32_5x5mm_Pitch0.5mm -> Housings_QFP:TQFP-32_7x7mm_Pitch0.8mm
- U1: symbol 7805 -> 7805-RESCUE-Tester
Changed lines of the file:
@@
 EESchema Schematic File Version 2
+LIBS:Tester-rescue
 LIBS:power
 LIBS:device
@@
 F 0 "IC1" H 3500 4150 40  0000 L BNN
 F 1 "ATMEGA328-A" H 4650 1500 40  0000 L BNN
-F 2 "Housings_QFP:LQFP-32_5x5mm_Pitch0.5mm" H 4250 2900 30  0000 C CIN
+F 2 "Housings_QFP:TQFP-32_7x7mm_Pitch0.8mm" H 4250 2900 30  0000 C CIN
 F 3 "" H 4250 2900 60  0000 C CNN
 	1    4250 2900
@@
 $EndComp
 $Comp
-L 7805 U1
+L 7805-RESCUE-Tester U1
 U 1 1 576E1991
 P 1650 1250

Commit message: Create Analog Sensor Board, Add Conglomerate1 Board (Advanced Circuits Order)
Parts:
- added C10, C11: 100n, Capacitors_SMD:C_1206, symbol C_Small
- added C9: 4.7u, Capacitors_SMD:C_1206, symbol C_Small
Connections:
- net +5V: now also C10.1, C11.1, C9.1
- net GND: now also C10.2, C11.2, C9.2
