File: Rocket Board/RocketBoard.sch (KiCad schematic (older format))
At the start: 52 parts, among them P1 PA_8, P10 PB_5, P11 PC_9, P12 PC_8, P13 PC_0, P14 PC_1, P15 PC_2, P16 PC_3, P17 CONN_01X04, P18 I2C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

Commit message: Partial Layout of Board
Started the board layout process
Parts:
- P17: value CONN_01X04 -> SWD
Connections:
- net PA_10: now also RP1.2 (P2); no longer RP1.3 (P3)
- net PA_11: now also RP1.1 (P1); no longer RP1.4 (P4)
- net PA_8: now also RP1.4 (P4); no longer RP1.1 (P1)
- net PA_9: now also RP1.3 (P3); no longer RP1.2 (P2)
Changed lines of the file:
@@
 P 6200 6200
 F 0 "P17" H 6200 6450 50  0000 C CNN
-F 1 "CONN_01X04" V 6300 6200 50  0000 C CNN
+F 1 "SWD" V 6300 6200 50  0000 C CNN
 F 2 "Pin_Headers:Pin_Header_Straight_1x04" H 6200 6200 60  0001 C CNN
 F 3 "" H 6200 6200 60  0000 C CNN
@@
 	1    0    0    -1
 $EndComp
-Text Label 2150 1200 2    60   ~ 0
+Text Label 2150 1500 2    60   ~ 0
 PA_8
 Text Label 1350 1550 0    60   ~ 0
 PA_8
-Text Label 2150 1300 2    60   ~ 0
+Text Label 2150 1400 2    60   ~ 0
 PA_9
 Text Label 1350 1650 0    60   ~ 0
 PA_9
-Text Label 2150 1400 2    60   ~ 0
+Text Label 2150 1300 2    60   ~ 0
 PA_10
 Text Label 1350 1750 0    60   ~ 0
 PA_10
-Text Label 2150 1500 2    60   ~ 0
+Text Label 2150 1200 2    60   ~ 0
 PA_11
 $Comp

Commit message: Fix analog input, Add 2 UART ports, changed PWM1/3 to PWM1/3N
Removed the series resistors for analog inputs, added pinouts for
UART1,2.   Changed PWM 1/3 tp PWM 1/3N to free up RX1 pin
Parts:
- removed RP4: 220 4pack, Resistors_SMD:R_Array_Convex_4x1206, symbol R_PACK4
- added UART1: UART1, Pin_Headers:Pin_Header_Straight_1x02, symbol CONN_01X02
- added UART2: UART2, Pin_Headers:Pin_Header_Straight_1x02, symbol CONN_01X02
- P1: value PA_8 -> PB_15
- P2: value PA_9 -> PB_11
- P3: value PA_10 -> PA_8
- P4: value PA_11 -> PA_9
Connections:
- net GND: no longer U1.16 (PA2), U1.17 (PA3), U1.36 (PB15), U1.58 (PB6)
- net PA_11: now also RP1.2 (P2); no longer RP1.1 (P1)
- net PC_0: now also P13.1 (P1)
- net PC_1: now also P14.1 (P1)
- net PC_2: now also P15.1 (P1)
- net PC_3: now also P16.1 (P1)
- net PA_10 renamed RX1
- net RX1: now also UART1.2 (P2); no longer RP1.2 (P2)
- new net PB_15: RP1.1 (P1), U1.36 (PB15)
- new net RX2: U1.17 (PA3), UART2.2 (P2)
- new net TX1: U1.58 (PB6), UART1.1 (P1)
- new net TX2: U1.16 (PA2), UART2.1 (P1)
Changed lines of the file:
@@
 P 3200 900
 F 0 "P1" H 3200 1050 50  0000 C CNN
-F 1 "PA_8" V 3300 900 50  0000 C CNN
+F 1 "PB_15" V 3300 900 50  0000 C CNN
 F 2 "Pin_Headers:Pin_Header_Straight_1x02" H 3200 900 60  0001 C CNN
 F 3 "" H 3200 900 60  0000 C CNN
@@
 P 3200 1950
 F 0 "P4" H 3200 2100 50  0000 C CNN
-F 1 "PA_11" V 3300 1950 50  0000 C CNN
+F 1 "PA_9" V 3300 1950 50  0000 C CNN
 F 2 "Pin_Headers:Pin_Header_Straight_1x02" H 3200 1950 60  0001 C CNN
 F 3 "" H 3200 1950 60  0000 C CNN
@@
 P 3200 1250
 F 0 "P2" H 3200 1400 50  0000 C CNN
-F 1 "PA_9" V 3300 1250 50  0000 C CNN
+F 1 "PB_11" V 3300 1250 50  0000 C CNN
 F 2 "Pin_Headers:Pin_Header_Straight_1x02" H 3200 1250 60  0001 C CNN
 F 3 "" H 3200 1250 60  0000 C CNN
@@
 P 3200 1600
 F 0 "P3" H 3200 1750 50  0000 C CNN
-F 1 "PA_10" V 3300 1600 50  0000 C CNN
+F 1 "PA_8" V 3300 1600 50  0000 C CNN
 F 2 "Pin_Headers:Pin_Header_Straight_1x02" H 3200 1600 60  0001 C CNN
 F 3 "" H 3200 1600 60  0000 C CNN
@@
 PA_9
 Text Label 2150 1300 2    60   ~ 0
-PA_10
-Text Label 1350 1750 0    60   ~ 0
-PA_10
-Text Label 2150 1200 2    60   ~ 0
 PA_11
 $Comp
@@
 	0    1    1    0
 $EndComp
-$Comp
-L R_PACK4 RP4
-U 1 1 5779A362
-P 4400 3300
-F 0 "RP4" H 4400 3750 50  0000 C CNN
-F 1 "220 4pack" H 4400 3250 50  0000 C CNN
-F 2 "Resistors_SMD:R_Array_Convex_4x1206" H 4400 3300 60  0001 C CNN
-F 3 "http://www.digikey.com/product-detail/en/yageo/YC164-JR-07220RL/YC164J-220CT-ND/1005664" H 4400 3300 60  0001 C CNN
-	1    4400 3300
-	1    0    0    -1
-$EndComp
 Text Notes 4400 2450 0    60   ~ 0
 Analog
@@
 	2700 3600 3050 3600
 Wire Wire Line
-	4600 2950 4700 2950
+	4200 2950 4700 2950
 Wire Wire Line
 	4700 2950 4700 2600
@@
 	4700 2600 5050 2600
 Wire Wire Line
-	4600 3050 4800 3050
+	4200 3050 4800 3050
 Wire Wire Line
 	4800 3050 4800 2950
@@
 	4800 2950 5050 2950
 Wire Wire Line
-	4600 3150 4800 3150
+	4200 3150 4800 3150
 Wire Wire Line
 	4800 3150 4800 3300
@@
 	4800 3300 5050 3300
 Wire Wire Line
-	4600 3250 4700 3250
+	4200 3250 4700 3250
 Wire Wire Line
 	4700 3250 4700 3650
@@
 	1700 4100 1350 4100
 Wire Wire Line
-	1700 4000 1350 4000
-Wire Wire Line
 	1700 2600 1700 4100
 Wire Wire Line
 	1700 3900 1350 3900
-Connection ~ 1700 4000
 Wire Wire Line
 	1350 3800 1700 3800
@@
 	1700 3300 1350 3300
 Connection ~ 1700 3600
-Wire Wire Line
-	1350 3200 1700 3200
 Connection ~ 1700 3300
 Wire Wire Line
 	1700 2900 1350 2900
-Connection ~ 1700 3200
 Wire Wire Line
 	1700 2600 1350 2600
@@
 $EndComp
 Wire Wire Line
-	1500 950  1500 1450
-Wire Wire Line
 	1500 1350 1350 1350
 Connection ~ 1500 1450
@@
 	1500 1150 1350 1150
 Connection ~ 1500 1250
-Wire Wire Line
-	1500 1050 1350 1050
 Connection ~ 1500 1150
-Wire Wire Line
-	1500 950  1350 950
-Connection ~ 1500 1050
 Text Label 1350 750  0    60   ~ 0
 PA_0
@@
 Wire Wire Line
 	6600 2300 6600 2150
+Wire Wire Line
+	1500 1150 1500 1450
+Text Label 1350 950  0    60   ~ 0
+TX2
+Text Label 1350 1050 0    60   ~ 0
+RX2
+Text Label 6400 3200 2    60   ~ 0
+TX2
+Text Label 6400 3300 2    60   ~ 0
+RX2
+$Comp
+L CONN_01X02 UART2
+U 1 1 57837830
+P 6750 3250
+F 0 "UART2" H 6750 3400 50  0000 C CNN
+F 1 "UART2" V 6850 3250 50  0000 C CNN
+F 2 "Pin_Headers:Pin_Header_Straight_1x02" H 6750 3250 60  0001 C CNN
+F 3 "" H 6750 3250 60  0000 C CNN
+	1    6750 3250
+	1    0    0    -1
+$EndComp
+Wire Wire Line
+	6400 3200 6550 3200
+Wire Wire Line
+	6400 3300 6550 3300
+Text Label 1350 3200 0    60   ~ 0
+TX1
+Text Label 1350 1750 0    60   ~ 0
+RX1
+Text Label 1350 4000 0    60   ~ 0
+PB_15
+Text Label 2150 1200 2    60   ~ 0
+PB_15
+Text Label 6400 3650 2    60   ~ 0
+TX1
+Text Label 6400 3750 2    60   ~ 0
+RX1
+$Comp
+L CONN_01X02 UART1
+U 1 1 5783FA1A
+P 6750 3700
+F 0 "UART1" H 6750 3850 50  0000 C CNN
+F 1 "UART1" V 6850 3700 50  0000 C CNN
+F 2 "Pin_Headers:Pin_Header_Straight_1x02" H 6750 3700 60  0001 C CNN
+F 3 "" H 6750 3700 60  0000 C CNN
+	1    6750 3700
+	1    0    0    -1
+$EndComp
+Wire Wire Line
+	6400 3650 6550 3650
+Wire Wire Line
+	6400 3750 6550 3750
 $EndSCHEMATC
